File: KiCAD/block-diagram/block-diagram-alex.kicad_sch (KiCad schematic)
At the start: 35 parts, among them J1 Conn_01x08, J2 Conn_01x08, J3 Conn_01x10, Q3 NMOS, Q4 NMOS, U1 74HC02, U3 74HC11, U6 LMC555xM

Commit message: Added Potentiometer Part number
Added part number and manufacturer number for the potentiometer.
Parts:
- RV1: CatNo (none) -> 987-1508-ND; MfgNo (none) -> 67YR50KLF
Changed lines of the file:
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@@
 			)
 		)
-		(property "CatNo" ""
-			(at 204.47 22.86 90)
+		(property "CatNo" "987-1508-ND"
+			(at 212.598 19.558 90)
 			(effects
 				(font
 					(size 1.27 1.27)
 				)
-				(hide yes)
 			)
 		)
-		(property "MfgNo" ""
+		(property "MfgNo" "67YR50KLF"
 			(at 204.47 22.86 90)
 			(effects

Commit message: Added Connector Part Numbers
Part and manufacturer number for connectors.
Parts:
- J1, J2, J3: CatNo (none) -> ED7264-10-ND; MfgNo (none) -> 800-10-010-10-001000
Changed lines of the file:
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@@
 			)
 		)
+		(property "CatNo" "ED7264-10-ND"
+			(at 274.32 125.984 0)
+			(effects
+				(font
+					(size 1.27 1.27)
+				)
+			)
+		)
+		(property "MfgNo" "800-10-010-10-001000"
+			(at 276.86 104.14 0)
+			(effects
+				(font
+					(size 1.27 1.27)
+				)
+				(hide yes)
+			)
+		)
 		(pin "7"
 		)
@@
 		(on_board yes)
 		(dnp no)
-		(fields_autoplaced yes)
 		(property "Reference" "J3"
 			(at 147.32 170.1799 0)
@@
 			)
 		)
+		(property "CatNo" "ED7264-10-ND"
+			(at 149.86 186.436 0)
+			(effects
+				(font
+					(size 1.27 1.27)
+				)
+			)
+		)
+		(property "MfgNo" "800-10-010-10-001000"
+			(at 144.78 170.18 0)
+			(effects
+				(font
+					(size 1.27 1.27)
+				)
+				(hide yes)
+			)
+		)
 		(pin "5"
 		)
@@
 		(on_board yes)
 		(dnp no)
-		(fields_autoplaced yes)
 		(property "Reference" "J1"
 			(at 101.6 69.85 0)
@@
 			(at 101.6 83.82 0)
 			(effects
+				(font
+					(size 1.27 1.27)
+				)
+				(hide yes)
+			)
+		)
+		(property "CatNo" "ED7264-10-ND"
+			(at 98.552 97.536 0)
+			(effects
+				(font
+					(size 1.27 1.27)
+				)
+			)
+		)
+		(property "MfgNo" "800-10-010-10-001000"
+			(at 101.6 83.82 0)
+			(effects

Commit message: Removed J3 part number
Removed the CatNo and MfgNo for J3
Parts:
- J3: CatNo ED7264-10-ND -> (none); MfgNo 800-10-010-10-001000 -> (none)
Changed lines of the file:
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@@
 			)
 		)
-		(property "CatNo" "ED7264-10-ND"
+		(property "CatNo" ""
 			(at 149.86 186.436 0)
 			(effects
@@
 					(size 1.27 1.27)
 				)
+				(hide yes)
 			)
 		)
-		(property "MfgNo" "800-10-010-10-001000"
+		(property "MfgNo" ""
 			(at 144.78 170.18 0)
 			(effects

Commit message: Set connector J3 to do not populate
Parts:
- J3: now not fitted
Changed lines of the file:
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@@
 		(in_bom yes)
 		(on_board yes)
-		(dnp no)
+		(dnp yes)
 		(property "Reference" "J3"
 			(at 147.32 170.1799 0)

Commit message: Fix missing 5V on schematic, update README
Connections:
- net +5V: now also C3.1, RV1.2, RV1.3, U6.8 (VCC)
Changed lines of the file:
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@@
+	)
+	(junction
+		(at 180.34 22.86)
+		(diameter 0)
+		(color 0 0 0 0)
 	)
 	(junction
@@
 	)
 	(junction
+		(at 184.15 22.86)
+		(diameter 0)
+		(color 0 0 0 0)
+	)
+	(junction
 		(at 271.78 106.68)
 		(diameter 0)
@@
 		)
 		(stroke
+			(width 0)
+			(type default)
+		)
+	)
+	(wire
+		(pts
+			(xy 180.34 22.86) (xy 184.15 22.86)
+		)
+		(stroke
